File: ECAD-Files/EAGLE-Files/Thanics Halo/Drone V2/Central Boardv2/Central Board.brd (EAGLE design)
At the start: 38.6 x 75.4 mm, 69 parts, among them J5 U.FL, J8 MICROSD, U3 LM3880MF-1AA/NOPBMF06A-M, U4 NEO-M8, U5 TPS6209, U7 MIC23050

Commit message: Started V3 Design
Connections:
- net GND: now also J4.6; no longer J4.9
- net GPCLK1: now also J4.9; no longer J4.6
Routing:
- net GPCLK1: track 47.8 -> 42.9 mm
- net GND: vias 44 -> 46
Other:
- board size 38.6 x 75.4 mm -> 38.5 x 75.3 mm
- board text added: "Central Board v4"
- board text removed: "Central Board v3"
Changed lines of the file:
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@@
 <?xml version="1.0" encoding="utf-8"?>
 <!DOCTYPE eagle SYSTEM "eagle.dtd">
-<eagle version="8.5.1">
+<eagle version="8.6.0">
 <drawing>
 <settings>
@@
 </layers>
 <board>
+<fusionsync huburn="a.cGVyc29uYWw6dWUyODQ3M2Rj" projecturn="a.cGVyc29uYWw6dWUyODQ3M2RjIzIwMTYxMDI3NDg3NTA0MzE" f3durn="urn:adsk.wipprod:dm.lineage:px5w3IuTSdeuRLXCAS-NGg" pcbguid="e94fe3bb-b015-404a-a45f-74c3c412db50" lastpulledtime="" lastsyncedchangeguid=""/>
 <plain>
-<wire x1="15.875" y1="0.1778" x2="54.5084" y2="0.0508" width="0" layer="20"/>
-<wire x1="15.9004" y1="75.3618" x2="15.875" y2="0.1778" width="0" layer="20"/>
 <hole x="52.8828" y="1.7018" drill="2.54"/>
-<text x="33.6804" y="31.8262" size="1.524" layer="25" rot="R90">Central Board v3</text>
-<wire x1="15.9004" y1="75.3618" x2="54.3814" y2="75.438" width="0" layer="20"/>
-<wire x1="54.3814" y1="75.438" x2="54.5084" y2="0.0508" width="0" layer="20"/>
+<text x="33.6804" y="31.8262" size="1.524" layer="25" rot="R90">Central Board v4</text>
 <hole x="17.5514" y="73.6346" drill="2.54"/>
 <wire x1="47.50775" y1="15.73505" x2="47.51001875" y2="15.740909375" width="0.0508" layer="25"/>
@@
 <text x="48.006" y="5.1308" size="1.27" layer="22" rot="MR270">J4</text>
 <text x="39.878" y="35.56" size="1.27" layer="22" rot="MR270">U7</text>
+<wire x1="15.9004" y1="0.1524" x2="54.4068" y2="0.1524" width="0" layer="20"/>
+<wire x1="54.4068" y1="0.1524" x2="54.4068" y2="75.438" width="0" layer="20"/>
+<wire x1="54.4068" y1="75.438" x2="15.9004" y2="75.438" width="0" layer="20"/>
+<wire x1="15.9004" y1="75.438" x2="15.9004" y2="0.1524" width="0" layer="20"/>
 </plain>
 <attributes>
@@
 <wire x1="18.6" y1="58.4708" x2="18.6298" y2="58.5006" width="0.1524" layer="1"/>
 <via x="32.004" y="73.8124" extent="1-16" drill="0.3048"/>
-<polygon width="0.254" layer="1">
+<polygon width="0.254" layer="1" rank="2">
 <vertex x="16.256" y="75.0824"/>
 <vertex x="54.4068" y="75.438"/>
@@
 <vertex x="16.256" y="0.0508"/>
 </polygon>
-<polygon width="0.254" layer="16">
+<polygon width="0.254" layer="16" rank="2">
 <vertex x="16.3068" y="75.1332"/>
 <vertex x="54.5084" y="75.3872"/>
@@
 <wire x1="35.12710625" y1="25.8572" x2="35.2552" y2="25.8572" width="0.1524" layer="16"/>
 <wire x1="33.91070625" y1="27.0736" x2="35.12710625" y2="25.8572" width="0.1524" layer="16"/>
-<contactref element="J4" pad="9"/>
 <via x="21.2852" y="65.4812" extent="1-16" drill="0.3048"/>
 <wire x1="20.9804" y1="66.8528" x2="20.701" y2="66.7258" width="0.1524" layer="1"/>
@@
 <wire x1="25.0444" y1="13.0048" x2="25.0444" y2="15.7988" width="0.1524" layer="16"/>
 <wire x1="25.0444" y1="15.7988" x2="24.892" y2="15.9512" width="0.1524" layer="16"/>
+<contactref element="J4" pad="6"/>
+<via x="37.846" y="14.3256" extent="1-16" drill="0.3048"/>
+<via x="43.434" y="11.2776" extent="1-16" drill="0.3048"/>
+<wire x1="18.6298" y1="27.9006" x2="18.6298" y2="29.7006" width="0" layer="19" extent="1-1"/>
 </signal>
 <signal name="N$1">
@@
 <signal name="GPCLK1">
 <contactref element="U6" pad="82"/>
-<contactref element="J4" pad="6"/>
 <wire x1="26.4298" y1="41.4006" x2="25.1954" y2="41.4006" width="0.1524" layer="1"/>
 <wire x1="25.1954" y1="41.4006" x2="25.0444" y2="41.2496" width="0.1524" layer="1"/>
@@
 <via x="35.5092" y="17.9832" extent="1-16" drill="0.3048"/>
 <wire x1="30.1752" y1="24.89965625" x2="30.1752" y2="23.3172" width="0.1524" layer="1"/>
-<via x="41.0464" y="16.002" extent="1-16" drill="0.3048"/>
-<via x="40.5892" y="11.3284" extent="1-16" drill="0.3048"/>
-<wire x1="40.624" y1="11.2936" x2="40.5892" y2="11.3284" width="0.1524" layer="16"/>
-<wire x1="40.624" y1="11.2936" x2="41.942" y2="11.2936" width="0.1524" layer="16"/>
-<wire x1="40.5892" y1="11.4808" x2="40.5892" y2="11.3284" width="0.1524" layer="1"/>
-<wire x1="37.8917" y1="16.002" x2="41.0464" y2="16.002" width="0.1524" layer="16"/>
+<wire x1="37.8917" y1="16.002" x2="39.2458" y2="16.002" width="0.1524" layer="16"/>
 <wire x1="37.8917" y1="16.002" x2="36.9265" y2="16.9672" width="0.1524" layer="16"/>
 <wire x1="36.9265" y1="16.9672" x2="36.5252" y2="16.9672" width="0.1524" layer="16"/>
 <wire x1="36.5252" y1="16.9672" x2="35.5092" y2="17.9832" width="0.1524" layer="16"/>
-<wire x1="41.0464" y1="16.002" x2="41.0464" y2="11.938" width="0.1524" layer="1"/>
-<wire x1="41.0464" y1="11.938" x2="40.5892" y2="11.4808" width="0.1524" layer="1"/>
 <wire x1="30.8102" y1="37.5666" x2="30.8102" y2="35.5346" width="0.1524" layer="16"/>
 <wire x1="30.8102" y1="35.5346" x2="29.7942" y2="34.5186" width="0.1524" layer="16"/>
 <contactref element="R10" pad="1"/>
-<wire x1="39.562396875" y1="12.355203125" x2="39.562396875" y2="13.1572" width="0.1524" layer="16"/>
-<wire x1="40.5892" y1="11.3284" x2="39.562396875" y2="12.355203125" width="0.1524" layer="16"/>
+<contactref element="J4" pad="9"/>
+<wire x1="39.2458" y1="16.002" x2="39.2684" y2="16.0246" width="0.1524" layer="16"/>
+<via x="39.2684" y="16.0246" extent="1-16" drill="0.35"/>
+<wire x1="39.2684" y1="16.0246" x2="40.132" y2="15.161" width="0.1524" layer="1"/>
+<wire x1="40.132" y1="15.161" x2="40.132" y2="14.478" width="0.1524" layer="1"/>
+<via x="40.132" y="14.478" extent="1-16" drill="0.35"/>
+<wire x1="40.132" y1="14.478" x2="40.3164" y2="14.2936" width="0.1524" layer="16"/>
+<wire x1="40.3164" y1="14.2936" x2="41.942" y2="14.2936" width="0.1524" layer="16"/>
+<wire x1="40.132" y1="14.478" x2="39.562396875" y2="13.908396875" width="0.1524" layer="16"/>
+<wire x1="39.562396875" y1="13.908396875" x2="39.562396875" y2="13.1572" width="0.1524" layer="16"/>
 </signal>
 <signal name="INT_A">
@@
 </board>
 </drawing>
+<compatibility>
+<note version="8.3" severity="warning">
+Since Version 8.3, EAGLE supports Fusion synchronisation.
+This feature will not be available in this version and saving
+the document will break the link to the Fusion PCB feature.
+</note>
+</compatibility>
 </eagle>
