File: ECAD-Files/EAGLE-Files/Thanics Halo/Drone V2/Flight Controller Auxiliary Board/Flight Controller Auxiliary Board.brd (EAGLE design)
At the start: 58.5 x 28.4 mm, 48 parts, among them J3 MAGJACK, U3 WGM110A

Commit message: Started V3 Design
Connections:
- net N$16: no longer J3.6
Routing:
- net GPCLK: track 5.76 -> 10.0 mm
- net RX_P: track 26.6 -> 28.7 mm
- net N$16: track 8.82 -> 7.21 mm
Other:
- outline, holes or cut-outs redrawn
