File: ECAD-Files/EAGLE-Files/Thanics Halo/Drone V2/Telemetry Transceiver Board/Telemetry Transceiver Board.brd (EAGLE design)
At the start: 31.4 x 41.1 mm, 5 parts

Commit message: Started V3 Design
Parts:
- renumbered U$1 to J1
Routing:
- net +3V3: track 31.2 -> 37.5 mm
- net TX: track 30.1 -> 30.9 mm, vias 2 -> 0
- net RX: vias 2 -> 0
Other:
- board text added: "J1"
Changed lines of the file:
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@@
 <?xml version="1.0" encoding="utf-8"?>
 <!DOCTYPE eagle SYSTEM "eagle.dtd">
-<eagle version="8.4.1">
+<eagle version="8.6.0">
 <drawing>
 <settings>
@@
 </layers>
 <board>
-<fusionsync huburn="a.cGVyc29uYWw6dWUyODQ3M2Rj" projecturn="a.cGVyc29uYWw6dWUyODQ3M2RjIzIwMTYxMDI3NDg3NTA0MzE" f3durn="urn:adsk.wipprod:dm.lineage:B3Psz0LATUywjwQQbWY99w" pcbguid="bc48e5cb-b012-4c9e-938b-b97e78c1de32" lastpulledtime="" lastsyncedchangeguid="65ac93e8-ac29-0601-ca15-8d0cffbec043"/>
+<fusionsync huburn="a.cGVyc29uYWw6dWUyODQ3M2Rj" projecturn="a.cGVyc29uYWw6dWUyODQ3M2RjIzIwMTYxMDI3NDg3NTA0MzE" f3durn="urn:adsk.wipprod:dm.lineage:ND8pgOG3TSSpkYMVTgUBdw" pcbguid="db24dc17-36a6-4ae4-bac8-4f72ddddcfb5" lastpulledtime="" lastsyncedchangeguid="eb3e9cff-90f1-c95d-b4ee-a542bdb51a0f"/>
 <plain>
 <wire x1="0" y1="-1.27" x2="31.42" y2="-1.27" width="0" layer="20"/>
@@
 <wire x1="31.42" y1="39.868" x2="0" y2="39.868" width="0" layer="20"/>
 <wire x1="0" y1="39.868" x2="0" y2="-1.27" width="0" layer="20"/>
-<hole x="2.794" y="37.338" drill="2.9972"/>
-<hole x="29.21" y="36.83" drill="2.9972"/>
+<hole x="2.54" y="37.338" drill="2.9972"/>
+<hole x="28.702" y="37.338" drill="2.9972"/>
 <hole x="29.464" y="0.762" drill="2.9972"/>
 <hole x="2.032" y="0.762" drill="2.9972"/>
@@
 Transceiver
 Board v1</text>
+<text x="19.558" y="36.068" size="1.778" layer="21">J1</text>
 </plain>
 <attributes>
@@
 <param name="checkRestrict" value="0"/>
 <param name="checkStop" value="0"/>
+<param name="checkValues" value="0"/>
 <param name="useDiameter" value="13"/>
 <param name="maxErrors" value="50"/>
@@
 <attribute name="OC_NEWARK" value="42M2667" x="15.572" y="16.366" size="1.778" layer="27" rot="R180" display="off"/>
 </element>
-<element name="U$1" library="thanics_robotics" package="JST_SH_4POS" value="" x="15.494" y="35.052"/>
+<element name="J1" library="thanics_robotics" package="JST_SH_4POS" value="" x="15.494" y="35.052"/>
 </elements>
 <signals>
@@
 <contactref element="XB1" pad="10"/>
 <contactref element="XB1" pad="14"/>
-<contactref element="U$1" pad="4"/>
+<contactref element="J1" pad="4"/>
 </signal>
 <signal name="+3V3">
@@
 <contactref element="XB1" pad="1"/>
 <contactref element="XB1" pad="5"/>
-<wire x1="26.572" y1="15.366" x2="26.798" y2="15.366" width="0.254" layer="1"/>
+<wire x1="26.798" y1="15.366" x2="26.572" y2="15.366" width="0.254" layer="1"/>
 <wire x1="26.798" y1="15.366" x2="28.194" y2="13.97" width="0.254" layer="1"/>
 <wire x1="28.194" y1="13.97" x2="28.194" y2="11.43" width="0.254" layer="1"/>
@@
 <wire x1="28.1813" y1="7.112" x2="26.826" y2="7.112" width="0.254" layer="1"/>
 <wire x1="26.826" y1="7.112" x2="26.572" y2="7.366" width="0.254" layer="1"/>
-<wire x1="13.994" y1="27.944" x2="26.572" y2="15.366" width="0.254" layer="1"/>
-<contactref element="U$1" pad="3"/>
-<wire x1="13.994" y1="27.944" x2="15.994" y2="35.052" width="0" layer="19" extent="1-1"/>
+<contactref element="J1" pad="3"/>
+<wire x1="26.572" y1="15.366" x2="15.994" y2="25.944" width="0.254" layer="1"/>
+<wire x1="15.994" y1="25.944" x2="15.994" y2="35.052" width="0.254" layer="1"/>
 </signal>
 <signal name="RX">
 <contactref element="XB1" pad="3"/>
-<wire x1="26.572" y1="11.366" x2="20.574" y2="17.364" width="0.254" layer="1"/>
-<contactref element="U$1" pad="2"/>
-<wire x1="20.574" y1="17.364" x2="20.574" y2="20.066" width="0.254" layer="1"/>
-<wire x1="20.574" y1="20.066" x2="14.986" y2="25.654" width="0.254" layer="1"/>
-<via x="14.986" y="25.654" extent="1-16" drill="0.35"/>
-<wire x1="14.986" y1="25.654" x2="14.986" y2="28.194" width="0.254" layer="16"/>
-<via x="14.986" y="28.194" extent="1-16" drill="0.35"/>
-<wire x1="14.986" y1="28.194" x2="14.986" y2="35.044" width="0.254" layer="1"/>
-<wire x1="14.986" y1="35.044" x2="14.994" y2="35.052" width="0.254" layer="1"/>
+<contactref element="J1" pad="2"/>
+<wire x1="26.572" y1="11.366" x2="14.994" y2="22.944" width="0.254" layer="1"/>
+<wire x1="14.994" y1="22.944" x2="14.994" y2="35.052" width="0.254" layer="1"/>
 </signal>
 <signal name="TX">
 <contactref element="XB1" pad="2"/>
-<wire x1="26.572" y1="9.366" x2="18.034" y2="17.904" width="0.254" layer="1"/>
-<wire x1="18.034" y1="17.904" x2="18.034" y2="19.304" width="0.254" layer="1"/>
-<wire x1="18.034" y1="19.304" x2="16.256" y2="21.082" width="0.254" layer="1"/>
-<via x="16.256" y="21.082" extent="1-16" drill="0.35"/>
-<wire x1="16.256" y1="21.082" x2="16.256" y2="33.528" width="0.254" layer="16"/>
-<wire x1="16.256" y1="33.528" x2="16.002" y2="33.782" width="0.254" layer="16"/>
-<via x="16.002" y="33.782" extent="1-16" drill="0.35"/>
-<wire x1="16.002" y1="33.782" x2="16.002" y2="35.044" width="0.254" layer="1"/>
-<contactref element="U$1" pad="1"/>
-<wire x1="16.002" y1="35.044" x2="13.994" y2="35.052" width="0" layer="19" extent="1-1"/>
+<contactref element="J1" pad="1"/>
+<wire x1="26.572" y1="9.366" x2="13.994" y2="21.944" width="0.254" layer="1"/>
+<wire x1="13.994" y1="21.944" x2="13.994" y2="35.052" width="0.254" layer="1"/>
 </signal>
 </signals>
