File: ECAD-Files/EAGLE-Files/Thanics Halo/Drone V3/PowerSwitchingBoard/PowerSwitchingBoard.brd (EAGLE design)
At the start: 80 x 88 mm, 248 parts, among them IC1 MEGA8-AI, IC3 MEGA8-AI, IC4 MEGA8-AI, IC5 MEGA8-AI, J1 ESC_CONTACTS, J3 62674-301121ALF, Q1 BC817, Q19 BC817, Q2 BC817, Q20 IRLR8726, Q21 IRLR8726, Q22 BC817, Q23 IRLR8726, Q24 IRLR8726, Q25 BC817, Q26 IRLR8726, Q27 IRLR8726, Q28 BC817, Q29 IRLR8726, Q3 BC817, Q30 IRLR8726, Q31 BC817, Q32 IRLR8726, Q33 IRLR8726, Q34 BC817, Q35 IRLR8726, Q36 IRLR8726, Q37 BC817, Q38 IRLR8726, Q39 IRLR8726, Q4 IRLR8726, Q40 BC817, Q41 IRLR8726, Q42 IRLR8726, Q43 BC817, Q44 IRLR8726, Q45 IRLR8726, Q5 IRLR8726, Q6 IRLR8726, Q7 IRLR8726, Q8 IRLR8726, Q9 IRLR8726, U1 TPS65261RHBR, U2 74HC4052PW, U3 74HC4052PW, U4 DRV8313, U5 DRV8313, U6 DRV8313, U7 74LVC1G10DW-7, U8 STM32F103RCT6LQFP-64-M, X1 16MHz, X3 16MHz, X4 16MHz, X5 16MHz, X6 8MHz

Commit message: Started routing programming traces
Parts:
- moved U3 202.0 mm to (43.7, 18.7), turned to 270 degrees
- moved J3 198.6 mm to (46.0, -0.38)
- moved U2 187.6 mm to (35.2, 16.1), turned to 270 degrees
- moved X6 180.3 mm to (51.9, 17.0), turned to 270 degrees
- moved J2 7.64 mm to (58.7, 4.19), turned to 90 degrees
- moved U8 4.70 mm to (60.8, 15.9)
- moved U7 4.16 mm to (31.9, 10.2)
- moved R144 2.32 mm to (46.4, 41.8)
- moved R145 2.32 mm to (46.4, 40.0)
- moved R37 2.22 mm to (33.8, 32.8)
- moved R38 2.22 mm to (33.8, 34.5)
- moved C42 1.48 mm to (44.2, 32.8), turned to 90 degrees
- moved C17 1.42 mm to (24.3, 14.7)
- moved C5 1.27 mm to (35.8, 41.7), turned to 270 degrees
- moved C31 1.26 mm to (44.3, 58.8), turned to 90 degrees
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Routing:
- net +5V: track 60.6 -> 134.2 mm, vias 0 -> 9
- net RST3: track 2.18 -> 44.2 mm, vias 0 -> 2
- net RST2: track 2.18 -> 41.1 mm
- net RST1: track 2.18 -> 38.7 mm, vias 0 -> 4
- net MOSI3: track 0.00 -> 35.7 mm
- net MISO3: track 0.00 -> 33.4 mm
- net SCK3: track 0.00 -> 31.2 mm
- net MOSI1: track 0.00 -> 30.0 mm, vias 0 -> 2
- net MOSI2: track 0.00 -> 25.6 mm
- net SCK2: track 0.00 -> 25.1 mm
- net MISO2: track 0.00 -> 24.7 mm
- net RESET: track 0.00 -> 23.2 mm
- net MISO1: track 0.00 -> 20.4 mm
- net MOSI4: track 0.00 -> 15.2 mm, vias 0 -> 2
- net MISO4: track 0.00 -> 11.3 mm, vias 0 -> 2
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
Commit message: Revert "Started routing programming traces"
This reverts commit 430756d4e182701a37896144ea8eedb7b4574f9e.
Parts:
- moved U3 202.0 mm to (-63.4, -152.7), turned to 0 degrees
- moved J3 198.6 mm to (-50.4, -174.0)
- moved U2 187.6 mm to (-63.4, -143.5), turned to 0 degrees
- moved X6 180.3 mm to (-58.8, -125.2), turned to 0 degrees
- moved J2 7.64 mm to (51.1, 4.70), turned to 180 degrees
- moved U8 4.70 mm to (56.1, 15.9)
- moved U7 4.16 mm to (28.3, 12.3)
- moved R144 2.32 mm to (44.1, 41.4)
- moved R145 2.32 mm to (44.1, 39.6)
- moved R37 2.22 mm to (35.9, 33.3)
- moved R38 2.22 mm to (35.9, 35.1)
- moved C42 1.48 mm to (43.4, 34.0), turned to 0 degrees
- moved C17 1.42 mm to (24.0, 13.3)
- moved C5 1.27 mm to (36.6, 40.6), turned to 180 degrees
- moved C31 1.26 mm to (43.4, 59.7), turned to 0 degrees
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Routing:
- net +5V: track 134.2 -> 60.6 mm, vias 9 -> 0
- net RST3: track 44.2 -> 2.18 mm, vias 2 -> 0
- net RST2: track 41.1 -> 2.18 mm
- net RST1: track 38.7 -> 2.18 mm, vias 4 -> 0
- net MOSI3: track 35.7 -> 0.00 mm
- net MISO3: track 33.4 -> 0.00 mm
- net SCK3: track 31.2 -> 0.00 mm
- net MOSI1: track 30.0 -> 0.00 mm, vias 2 -> 0
- net MOSI2: track 25.6 -> 0.00 mm
- net SCK2: track 25.1 -> 0.00 mm
- net MISO2: track 24.7 -> 0.00 mm
- net RESET: track 23.2 -> 0.00 mm
- net MISO1: track 20.4 -> 0.00 mm
- net MOSI4: track 15.2 -> 0.00 mm, vias 2 -> 0
- net MISO4: track 11.3 -> 0.00 mm, vias 2 -> 0
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