File: ECAD-Files/EAGLE-Files/Thanics Halo/Controller/Controller Board/Controller Board.sch (EAGLE design)
At the start: 154 parts, among them J10 EDGE_CONNECTOR_20POS, J2 3.5_TOUCHSCREEN, J3 USB_MICRO_B_SMT, J5 EDGE_CONNECTOR_20POS, J6 POWER_CONNECTOR, J7 HDMI, J8 2_PIN_CONNECTOR, J9 USB_A_RECEPT, Q2 2N7002P_MOSFET, U1 AAT3620_BATT_CHARGER, U10 TPS6209, U11 LM3880MF-1AA/NOPBMF06A-M, U12 APPLE_2.0C_COPROCESSOR, U16 MIC23050, U19 WM8960, U2 8 CH, U7 ESD5384, U8 PEC12R, U9 PEC12R, Y1 DSC6001

Commit message: About to remove touchscreen from controller board
Parts:
- added C42: 22uF, 22uF X5R Ceramic Capacitor:GRM21BR60J226ME39L
- added C43: 10uF, 10uF X5R Ceramic Capacitor:GRM21BR60J106ME19L
- added D5, D7: GREEN, SparkFun-LED:LED-GREEN0603
- added R22, R34: 1k, 1k-resistor:RC0603JR-071KLRC0603N-M
- added R35: 10k, 10k-resistor(0603):RC0603JR-0710KLRC0603N-M
- added U4: PDDL2450, thanics_robotics:PDDL2450
Connections:
- new net ETH_BIAS: U4.ETH_BIAS
- new net GND2: D5.C, U4.LINK_LED_LAN
- new net N$66: D5.A, R22.11
- new net N$67: R35.22, U4.CONFIG
- new net N$68: D7.A, U4.CPU_STAT_LED
- new net N$69: D7.C, R34.11
- new net RX_LAN_N: U4.RX_N_LAN
- new net RX_LAN_P: U4.RX_P_LAN
- new net TX_LAN_N: U4.TX_N_LAN
- new net TX_LAN_P: U4.TX_P_LAN
- net +3V3: now also C43.11, R35.11, U4.VCC, U4.VCC@2
- net +5V: now also C42.11, U4.VRF, U4.VRF@2
- net 3.3V_A: now also R22.22
- net GND: now also C42.22, C43.22, R34.22, U4.65, U4.66, U4.67, U4.68, U4.69, U4.70, U4.71, U4.72, U4.73, U4.74, U4.75, U4.76, U4.77, U4.78, U4.79, U4.80, U4.GND, U4.GND@2, U4.GND@3, U4.GND@4, U4.GND@5, U4.GND@6
Other:
- note removed: "21-DIN 19-WCLK 18-BCLK"
- moved on the sheet: C20, C21, C22, C23, C24, C25, C26, C27, C28, C29, C30, C31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

Commit message: Finished controller board v1.5
Parts:
- removed J11: (no value), thanics_robotics:JST_SH_4POS
- removed JP2: (no value), Controller Board:PINHD-1X3
- removed Q5, Q6: (no value), Controller Board:DMG1012T
- removed R31: 20R, Controller Board:RC0603JR-0720RLRC0603N-M
- removed R38: NF, Controller Board:ERA-6AEB103V
- removed R39: 100k, Controller Board:RC0603JR-07100KLRC0603N-M
- removed R4: 10k, Controller Board:ERA-6AEB103V
- removed U$2: MICROSD, Controller Board:MICROSD
- removed U18: (no value), Controller Board:ESP12ESMD
- added C44, C45, C46, C47, C51, C52, C56, C69: 0.1uF, 0.1uF-capacitor-0402:0402ZD104KAT2A0402-M
- added C48: 1uF, thanics-capacitor:CL05A105MP5NNNC
- added C49, C50: 22uF, thanics-capacitor:CL21A226MOCLRNC
- added F1, F2, F3: MFU0603FF01600P100, 1.6a-fuse:MFU0603FF01600P100
- added L4: 1k@100MHz, 600ohm-fb:BLM18AG601SN1DIND_BLM18_0603-M
- added R36, R37, R44, R46, R47, R53, R54, R55: 49R9, 49.9-resistor:RC0402FR-0749K9LRC0402N-M
- added T1, T2: ALT4532M, thanics_robotics:ALT4532M
- C3: value 1uF -> 1uF; device Controller Board:CC0805KKX7R7BB105 -> thanics-capacitor:CL05A105MP5NNNC
- C35: device Controller Board:08055C104KAT2A -> 0.1uF-capacitor-0402:0402ZD104KAT2A0402-M
- C53: value 1uF -> 0.1uF; device 1uF X7R Ceramic Capacitor:CC0805KKX7R7BB105 -> 0.1uF-capacitor-0402:0402ZD104KAT2A0402-M
- J2: value 3.5_TOUCHSCREEN -> USB_A_RECEPT; device Controller Board:3.5_TOUCHSCREEN -> Controller Board:USB_A_RECEPT
- J3: value USB_MICRO_B_SMT -> 105450-0101; device Controller Board:USB_MICRO_B_SMT -> 105450-0101:105450-0101
- J6: value POWER_CONNECTOR -> MICROSD; device Controller Board:POWER_CONNECTOR -> Controller Board:MICROSD
- J7: value HDMI -> 105450-0101; device Controller Board:HDMI -> 105450-0101:105450-0101
- J9: value USB_A_RECEPT -> B2B-PH-SM4-TB(LF)(SN); device Controller Board:USB_A_RECEPT -> thanics-connector:B2B-PH-SM4-TB(LF)(SN)
- R1: value 100 -> 10k; device Controller Board:100_RESISTOR -> 10k-resistor(0603):RC0603JR-0710KLRC0603N-M
- R10, R16, R2, R23, R24, R25, R26, R27, R28, R29, R41, R45, R5, R8, R9: device Controller Board:ERA-6AEB103V -> 10k-resistor(0603):RC0603JR-0710KLRC0603N-M
- R11, R15: value 20R -> 22k; device Controller Board:RC0603JR-0720RLRC0603N-M -> thanics-resistor:RMCF0603JT22K0
- R14: value 20R -> 5.1k; device Controller Board:RC0603JR-0720RLRC0603N-M -> thanics-resistor:RMCF0603JT5K10
- R17: value 20R -> 1k; device Controller Board:RC0603JR-0720RLRC0603N-M -> 1k-resistor:RC0603JR-071KLRC0603N-M
- R18: value 340R -> 1k; device Controller Board:RC0603FR-07340RL -> 1k-resistor:RC0603JR-071KLRC0603N-M
- R19: value 24.9k -> 100R; device Controller Board:RC0402FR-0724K9LRC0402N-M -> 100-resistor:RC0603JR-07100RLRC0603N-M
- R21: value 20R -> 10k; device Controller Board:RC0603JR-0720RLRC0603N-M -> 10k-resistor(0603):RC0603JR-0710KLRC0603N-M
- R3: value 100k -> 5.1k; device Controller Board:RC0603JR-07100KLRC0603N-M -> thanics-resistor:RMCF0603JT5K10
- R30: value 20R -> 75k; device Controller Board:RC0603JR-0720RLRC0603N-M -> thanics-resistor:RMCF0603JT75K0
- R51: device 10k-resistor:ERA-6AEB103V -> 10k-resistor(0603):RC0603JR-0710KLRC0603N-M
- U11: value LM3880MF-1AA/NOPBMF06A-M -> (none); device Controller Board:LM3880MF-1AA/NOPBMF06A-M -> ICM-20948-mpu:ICM-20948
- U7: value ESD5384 -> (none); device Controller Board:ESD5384 -> thanics_robotics:FXMAR2102
Connections:
- removed net EMMC_EN_N_1V8: U6.EMMC_EN_N_1V8
- removed net HDMI_HPD_N_1V8: Q5.D, R39.22, U6.HDMI_HPD_N_1V8
- removed net IRQ: J2.GPIO25, U6.GPIO40
- removed net N$25: R15.11, U18.*GPIO9
- removed net N$26: R21.11, U18.*GPIO10
- removed net N$27: R30.11, U18.MOSI
- removed net N$40: JP2.1, R3.22
- removed net N$42: JP2.3, R19.22
- removed net N$8: R48.22, U10.EN, U11.FLAG1
- removed net POWER_SEQ_EN: R4.22, U11.EN
- new net I2C_SCL_1V8: U11.SCL/SCLK, U7.B0
- new net I2C_SDA_1V8: U11.SDA/SDI, U7.B1
- new net N$47: F1.1, J3.VBUS@1, J3.VBUS@2, J3.VBUS@3, J3.VBUS@4
- new net N$51: C50.1, F2.1, J7.VBUS@1, J7.VBUS@2, J7.VBUS@3, J7.VBUS@4
- new net N$63: J7.CC2, R15.1
- new net N$70: C45.2, C46.2, L4.1, R47.11, R53.11, R54.11, R55.11, T1.6, T2.6
- new net N$71: F3.2, J2.VCC
- net +1V8: now also C51.1, C52.2, C69.1, U11.AD0/SDO, U11.CS, U11.VDD, U11.VDDIO, U7.VCCB; no longer R39.11
- net +3V3: now also C56.2, J6.VDD, U7.OE, U7.VCCA; no longer C35.2, J11.2, R38.11, U$2.VDD, U18.VCC
- net +5V: now also C49.1, F2.2, F3.1, R11.2, R15.2; no longer J2.5V, J9.VCC, Q6.G, U7.5V, U7.RPU, U7.RPU2
- net 3.3V_A: now also C47.2, R36.11, R37.11, R44.11, R46.11, T1.3, T2.3; no longer J10.1
- net BATT_OUTPUT: now also R48.22; no longer R4.11, R48.11, U11.VCC
- net ETH_BIAS: now also C44.2, L4.2
- net GND: now also C3.2, C44.1, C45.1, C46.1, C47.1, C48.2, C49.2, C50.2, C51.2, C52.1, C53.1, C56.1, C69.2, J3.GND@1, J3.GND@2, J3.GND@3, J3.GND@4, J3.SHIELD, J6.VSS, J7.SHIELD, J9.2, R1.22, R14.1, R21.22, R3.1, R30.1, U11.FSYNC; no longer C3.1, C53.11, J11.1, J3.GND, J3.ID, J6.GND, J7.GND@5, J7.GND@6, J7.GND@7, J7.GND@8, J7.GND@9, J9.GND, Q5.S, R19.11, R3.11, U$2.VSS, U18.GND, U7.GND@2
- net HDMI_CEC: no longer Q6.S, R38.22
- net HDMI_CK_N: no longer J7.CLK_N
- net HDMI_CK_P: no longer J7.CLK_P
- net HDMI_D0_N: no longer J7.TX0_N
- net HDMI_D0_P: no longer J7.TX0_P
- net HDMI_D1_N: no longer J7.TX1_N
- net HDMI_D1_P: no longer J7.TX1_P
- net HDMI_D2_N: no longer J7.TX2_N
- net HDMI_D2_P: no longer J7.TX2_P
- net HDMI_SCL: no longer J7.SCL, U7.SCL
- net HDMI_SDA: no longer J7.SDA, U7.SDA
- net I2C_SCL: now also U7.A0; no longer J11.4
- net I2C_SDA: now also U7.A1; no longer J11.3
- net ID_SD: no longer U18.CH_PD
- net ISET: now also R30.2; no longer JP2.2
- net J2_SW: now also U6.GPIO41; no longer U6.GPIO39
- net N$12: now also C35.2, R48.11; no longer R49.22, U11.FLAG2
- net N$3: now also R49.22, U10.EN; no longer R14.11, U18.MISO
- net N$46: now also J3.CC2, R14.2; no longer R31.11, U18.SCLK
- net N$49: now also J3.CC1, R3.2; no longer J7.CEC_DAT, Q6.D, U7.CEC
- net N$50: now also J7.CC1, R11.1; no longer J7.HPD, Q5.G, U7.HPD
- net N$59: now also C48.1; no longer C53.22
- net N$6: now also C3.1, R19.22; no longer C3.2, R1.11
- net N$7: now also C53.2, U11.REGOUT; no longer R11.11, U18.CS0
- net RX_LAN_N: now also R54.22, T1.1
- net RX_LAN_P: now also R53.22, T1.2
- net RX_N: now also R46.22, T1.5; no longer J10.15
- net RX_P: now also R44.22, T1.4; no longer J10.16
- net SDX_CLK: now also J6.CLK; no longer U$2.CLK
- net SDX_CMD: now also J6.CMD; no longer U$2.CMD
- net SDX_D0: now also J6.DAT0; no longer U$2.DAT0
- net SDX_D1: now also J6.DAT1; no longer U$2.DAT1
- net SDX_D2: now also J6.DAT2; no longer U$2.DAT2
- net SDX_D3: now also J6.CD/DAT3; no longer U$2.CD/DAT3
- net SD_CLK: no longer R31.22
- net SD_CMD: no longer R11.22
- net SD_D0: no longer R14.22
- net SD_D1: no longer R30.22
- net SD_D2: no longer R15.22
- net SD_D3: no longer R21.22
- net SPI_CS0: no longer J2.CS0
- net SPI_CS1: no longer J2.CS1
- net SPI_MISO: no longer J2.MISO
- net SPI_MOSI: no longer J2.MOSI
- net SPI_SCLK: no longer J2.SCLK
- net STAT1: now also R1.11
- net STAT2: now also R21.11
- net SWITCH_IN: now also J9.1; no longer J6.5V
- net TX_LAN_N: now also R47.22, T2.1
- net TX_LAN_P: now also R55.22, T2.2
- net TX_N: now also R37.22, T2.5; no longer J10.12
- net TX_P: now also R36.22, T2.4; no longer J10.13
- net USB_5V: now also F1.2, R19.11; no longer J3.VCC, R1.22
- net USB_D2_N: now also J7.D-@1, J7.D-@2; no longer J9.D-
- net USB_D2_P: now also J7.D+@1, J7.D+@2; no longer J9.D+
- net USB_D3_N: now also J2.D-
- net USB_D3_P: now also J2.D+
Other:
- note added: "Logic Shifting"
- note added: "Sensors"
- note removed: "Charge Current Set: 1-2 = 2A Charge 2-3 = 500mA Charge"
- note removed: "HDMI"
- moved on the sheet: C53, C8, D4, R1, R19, R21, R33, R41, R48, R49, U12

Commit message: Added new battery and joystick modules
Parts:
- removed C33: 10uF, Controller Board:GRM21BR60J106ME19L
- removed U3: (no value), Controller Board:TPS61256YFFR
- added C70: 22uF, Controller Board:GRM21BR60J226ME39L
- added R31, R4: 10k, 10k-resistor(0603):RC0603JR-0710KLRC0603N-M
- added U13: MIC2876UDFN-8, thanics_robotics:MIC2876UDFN-8
Connections:
- net +3V3: now also J10.11; no longer J10.2
- net +5V: now also C70.2, U13.OUT, U13.OUTS; no longer C33.2, U3.VOUT
- net BATT_OUTPUT: now also U13.EN, U13.IN; no longer U3.EN, U3.VIN
- net GND: now also C70.1, J10.15, R31.22, R4.22, U13.AGND, U13.PGND; no longer C33.1, J10.11, J10.14, J10.17, U3.GND
- net J1_SW: now also R4.11
- net J2_SW: now also J10.12, R31.11; no longer J10.18
- net N$19: now also J10.13; no longer J10.19
- net N$20: now also J10.14; no longer J10.20
- net N$61: now also U13.SW; no longer U3.SW
Other:
- moved on the sheet: L1
