File: ECAD-Files/EAGLE-Files/Thanics Halo/Controller/Joystick Module B/Joystick Module B.sch (EAGLE design)
At the start: 2 parts

Commit message: Added new battery and joystick modules
Parts:
- removed U$3: JOYSTICK", thanics_robotics:JOYSTICK"
- added SW1: 2-1825910-7, spst-tactile-switch:2-1825910-7
- added U1: 27800-JOYSTICK, thanics_robotics:27800-JOYSTICK
Connections:
- net +3V3: now also SW1.1, U1.3V3; no longer U$3.3V3
- net GND: now also U1.GND; no longer U$3.GND
- net J2_SW: now also SW1.3; no longer U$3.SW
- net VRX: now also U1.VRX; no longer U$3.VRX
- net VRY: now also U1.VRY; no longer U$3.VRY
Changed lines of the file:
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@@
 <?xml version="1.0" encoding="utf-8"?>
 <!DOCTYPE eagle SYSTEM "eagle.dtd">
-<eagle version="8.4.1">
+<eagle version="9.0.0">
 <drawing>
 <settings>
@@
 <layers>
 <layer number="1" name="Top" color="4" fill="1" visible="no" active="no"/>
+<layer number="2" name="Route2" color="1" fill="3" visible="no" active="no"/>
+<layer number="15" name="Route15" color="4" fill="6" visible="no" active="no"/>
 <layer number="16" name="Bottom" color="1" fill="1" visible="no" active="no"/>
 <layer number="17" name="Pads" color="2" fill="1" visible="no" active="no"/>
@@
 </classes>
 <parts>
-<part name="U$3" library="thanics_robotics" deviceset="JOYSTICK" device="&quot;"/>
 <part name="U$1" library="thanics_robotics" deviceset="EDGE_CONNECTOR_20POS_CONTACTS" device=""/>
 <part name="+3V1" library="supply1" deviceset="+3V3" device=""/>
@@
 <part name="GND2" library="supply1" deviceset="GND" device=""/>
 <part name="+3V2" library="supply1" deviceset="+3V3" device=""/>
+<part name="U1" library="thanics_robotics" deviceset="27800-JOYSTICK" device=""/>
+<part name="SW1" library="spst-tactile-switch" deviceset="2-1825910-7" device=""/>
+<part name="+3V3" library="supply1" deviceset="+3V3" device=""/>
 </parts>
 <sheets>
@@
 </plain>
 <instances>
-<instance part="U$3" gate="A" x="-53.34" y="20.32"/>
 <instance part="U$1" gate="G$1" x="-63.5" y="-33.02"/>
 <instance part="+3V1" gate="G$1" x="-38.1" y="-15.24"/>
@@
 <instance part="GND2" gate="1" x="-38.1" y="10.16"/>
 <instance part="+3V2" gate="G$1" x="-38.1" y="33.02"/>
+<instance part="U1" gate="A" x="-53.34" y="20.32"/>
+<instance part="SW1" gate="A" x="-124.46" y="-2.54"/>
+<instance part="+3V3" gate="G$1" x="-127" y="7.62"/>
 </instances>
 <busses>
@@
 </segment>
 <segment>
-<pinref part="U$3" gate="A" pin="SW"/>
-<wire x1="-43.18" y1="22.86" x2="-33.02" y2="22.86" width="0.1524" layer="91"/>
-<label x="-40.64" y="22.86" size="1.778" layer="95"/>
+<pinref part="SW1" gate="A" pin="3"/>
+<wire x1="-86.36" y1="-2.54" x2="-71.12" y2="-2.54" width="0.1524" layer="91"/>
+<label x="-83.82" y="-2.54" size="1.778" layer="95"/>
 </segment>
 </net>
@@
 </segment>
 <segment>
-<pinref part="U$3" gate="A" pin="VRX"/>
 <wire x1="-43.18" y1="20.32" x2="-33.02" y2="20.32" width="0.1524" layer="91"/>
 <label x="-40.64" y="20.32" size="1.778" layer="95"/>
+<pinref part="U1" gate="A" pin="VRX"/>
 </segment>
 </net>
@@
 </segment>
 <segment>
-<pinref part="U$3" gate="A" pin="VRY"/>
 <wire x1="-43.18" y1="17.78" x2="-33.02" y2="17.78" width="0.1524" layer="91"/>
 <label x="-40.64" y="17.78" size="1.778" layer="95"/>
+<pinref part="U1" gate="A" pin="VRY"/>
 </segment>
 </net>
@@
 </segment>
 <segment>
-<pinref part="U$3" gate="A" pin="3V3"/>
 <wire x1="-43.18" y1="25.4" x2="-38.1" y2="25.4" width="0.1524" layer="91"/>
 <wire x1="-38.1" y1="25.4" x2="-38.1" y2="30.48" width="0.1524" layer="91"/>
 <pinref part="+3V2" gate="G$1" pin="+3V3"/>
+<pinref part="U1" gate="A" pin="3V3"/>
+</segment>
+<segment>
+<pinref part="SW1" gate="A" pin="1"/>
+<pinref part="+3V3" gate="G$1" pin="+3V3"/>
+<wire x1="-121.92" y1="-2.54" x2="-127" y2="-2.54" width="0.1524" layer="91"/>
+<wire x1="-127" y1="-2.54" x2="-127" y2="5.08" width="0.1524" layer="91"/>
 </segment>
 </net>
@@
 </segment>
 <segment>
-<pinref part="U$3" gate="A" pin="GND"/>
 <wire x1="-43.18" y1="15.24" x2="-38.1" y2="15.24" width="0.1524" layer="91"/>
 <wire x1="-38.1" y1="15.24" x2="-38.1" y2="12.7" width="0.1524" layer="91"/>
 <pinref part="GND2" gate="1" pin="GND"/>
-</segment>
-</net>
+<pinref part="U1" gate="A" pin="GND"/>
+</segment>
+</net>
